File: Power_Board_V2/MOSAIC Power Board.kicad_pcb (KiCad board)
At the start: 2 copper layers, 89 x 89 mm, 106 parts, among them J1 CONN 2MM JST, J10 CONN 2MM JST, J11 CONN 2MM JST, J12 CONN 2MM JST, J15 CONN 2MM JST, J16 CONN 2MM JST, J2 CONN 2MM JST, J3 CONN 2MM JST, J4 CONN 2MM JST, J5 CONN 2MM JST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

Commit message: routing work
Parts:
- removed JP1, JP10, JP11, JP12, JP13, JP14, JP15, JP16, JP17, JP18, JP19, JP2, JP8, JP9: SolderJumper_2_Open, Jumper:SolderJumper-2_P1.3mm_Open_RoundedPad1.0x1.5mm
- removed R10, R11, R13, R14, R16, R17, R19, R2, R20, R22, R23, R27, R28, R3: 10 kOhm, power_board_footprints_V2.0:R_0805
- added LOGO3: ~, power_board_footprints_V2.0:QWIIC_logo_8MM, F.Cu at (241.0, 88.0)
- D13, D14, J15, R26, TP3, TP6, U8: moved to B.Cu
- moved TP2 181.1 mm to (184.5, 124.2), turned to -90 degrees
- moved TP4 174.3 mm to (184.5, 105.2), turned to -90 degrees
- moved J14 173.6 mm to (175.5, 88.0), turned to -90 degrees
- moved TP6 172.1 mm to (184.5, 98.3), turned to 90 degrees
- moved TP7 170.9 mm to (184.2, 72.5), turned to -90 degrees
- moved LED1 161.1 mm to (180.7, 74.8)
- moved LOGO2 159.9 mm to (179.0, 88.0), turned to -90 degrees
- moved R25 159.7 mm to (179.2, 77.0)
- moved U9 159.4 mm to (177.1, 79.9), turned to -90 degrees
- moved C3 159.1 mm to (174.2, 80.0), turned to -90 degrees
- moved D4 158.7 mm to (201.4, 131.0), turned to 180 degrees
- moved U8 156.3 mm to (197.3, 59.9), turned to 90 degrees
- moved R24 156.0 mm to (182.2, 77.2), turned to 90 degrees
- moved D12 155.9 mm to (201.5, 118.6), turned to 180 degrees
- moved D8 155.8 mm to (201.5, 106.1), turned to 180 degrees
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Connections:
- J13 pad 3: /SD0 -> /SDA
- J13 pad 4: /SC0 -> /SCL
- J14 pad 3: /SD0 -> /SDA
- J14 pad 4: /SC0 -> /SCL
- R4 pad 2: /SD0 -> /SDA
- R5 pad 2: /SC0 -> /SCL
- U1 pad 1: Net-(JP2-A) -> unconnected-(U1-A1-Pad1)
- U1 pad 2: Net-(JP1-A) -> unconnected-(U1-A0-Pad2)
- U2 pad 1: Net-(JP8-A) -> unconnected-(U2-A1-Pad1)
- U2 pad 2: Net-(JP9-A) -> unconnected-(U2-A0-Pad2)
- U2 pad 3: /SD0 -> /SD1
- U2 pad 4: /SC0 -> /SC1
- U3 pad 1: Net-(JP10-A) -> unconnected-(U3-A1-Pad1)
- U3 pad 2: Net-(JP11-A) -> unconnected-(U3-A0-Pad2)
- U3 pad 3: /SD0 -> /SD2
- U3 pad 4: /SC0 -> /SC2
- U4 pad 1: Net-(JP12-A) -> unconnected-(U4-A1-Pad1)
- U4 pad 2: Net-(JP13-A) -> unconnected-(U4-A0-Pad2)
- U4 pad 3: /SD0 -> /SD3
- U4 pad 4: /SC0 -> /SC3
- U5 pad 1: Net-(JP14-A) -> unconnected-(U5-A1-Pad1)
- U5 pad 2: Net-(JP15-A) -> unconnected-(U5-A0-Pad2)
- U5 pad 3: /SD0 -> /SD4
- U5 pad 4: /SC0 -> /SC4
- U6 pad 1: Net-(JP16-A) -> unconnected-(U6-A1-Pad1)
- U6 pad 2: Net-(JP17-A) -> unconnected-(U6-A0-Pad2)
- U6 pad 3: /SD0 -> /SD5
- U6 pad 4: /SC0 -> /SC5
- U7 pad 10: /SD0 -> /SD3
- U7 pad 11: /SC0 -> /SC3
- U7 pad 13: /SD0 -> /SD4
- U7 pad 14: /SC0 -> /SC4
- U7 pad 15: /SD0 -> /SD5
- U7 pad 16: /SC0 -> /SC5
- U7 pad 17: /SD0 -> /SD6
- U7 pad 18: /SC0 -> /SC6
- U7 pad 6: /SD0 -> /SD1
- U7 pad 7: /SC0 -> /SC1
- U7 pad 8: /SD0 -> /SD2
- U7 pad 9: /SC0 -> /SC2
- U8 pad 1: Net-(JP18-A) -> unconnected-(U8-A1-Pad1)
- U8 pad 2: Net-(JP19-A) -> unconnected-(U8-A0-Pad2)
- U8 pad 3: /SD0 -> /SD6
- U8 pad 4: /SC0 -> /SC6
Routing:
- net VIN: track 0.00 -> 162.5 mm, vias 0 -> 4
- net /solar_IN: track 0.00 -> 160.4 mm, vias 0 -> 4
- net /SCL: track 0.00 -> 114.8 mm, vias 0 -> 8
- net /SDA: track 0.00 -> 106.6 mm, vias 0 -> 4
- net V_BATT: track 0.00 -> 97.6 mm, vias 0 -> 4
- net /SD0: track 0.00 -> 84.6 mm, vias 0 -> 4
- net /SC0: track 0.00 -> 78.1 mm, vias 0 -> 4
- net /SD1: track 0.00 -> 61.2 mm, vias 0 -> 2
- net /SC1: track 0.00 -> 56.8 mm
- net /SD4: track 0.00 -> 50.4 mm, vias 0 -> 2
- net /SD2: track 0.00 -> 50.3 mm, vias 0 -> 4
- net /SC4: track 0.00 -> 49.8 mm, vias 0 -> 2
- net /SD5: track 0.00 -> 49.1 mm, vias 0 -> 2
- net /SD6: track 0.00 -> 48.5 mm, vias 0 -> 3
- net /SC2: track 0.00 -> 47.4 mm, vias 0 -> 4
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Other:
- board text added: "A0"
- board text added: "A1"
- board text added: "I2C Multiplexer"
- board text added: "Main Board"

Commit message: finished v2.0
Parts:
- moved REF** 91.9 mm to (184.5, 136.0)
- moved LOGO1 48.0 mm to (235.5, 136.0)
Routing:
- net VIN: track 162.5 -> 233.8 mm, vias 4 -> 6
- net GND: track 0.00 -> 57.1 mm, vias 0 -> 35
- net Net-(JP6-B): track 5.63 -> 8.48 mm
Other:
- board text added: "Batt"
- board text added: "Batt IN"
- board text added: "I2C Address: 0x70"
- board text added: "Multiplexer Table"
- board text added: "SD0/SC0"
- board text added: "SD1/SC1"
- board text added: "SD2/SC2"
- board text added: "SD3/SC3"
- board text added: "SD4/SC4"
- board text added: "SD5/SC5"
- board text added: "SD6/SC6"
