File: Power_Board_V2/MOSAIC Power Board.kicad_sch (KiCad schematic)
At the start: 21 parts, among them J1 CONN 2MM JST, J10 CONN 2MM JST, J11 CONN 2MM JST, J12 CONN 2MM JST, J2 CONN 2MM JST, J3 CONN 2MM JST, J4 CONN 2MM JST, J5 CONN 2MM JST, J6 CONN 2MM JST, J7 CONN 2MM JST, J8 CONN 2MM JST, J9 CONN 2MM JST, U1 INA219AIDR, U2 TCA9548APWR

Commit message: work on schematic
Parts:
- added JP3, JP4: SolderJumper_2_Bridged, Jumper:SolderJumper-2_P1.3mm_Bridged_RoundedPad1.0x1.5mm, symbol Jumper:SolderJumper_2_Bridged
- added JP5, JP6, JP7: SolderJumper_2_Open, Jumper:SolderJumper-2_P1.3mm_Open_RoundedPad1.0x1.5mm, symbol Jumper:SolderJumper_2_Open
- added R4, R5, R6, R7, R8: 10 kOhm, power_board_footprints_V2.0:R_0805, symbol power_board_symbols_V2.0:R_10kOhm_1/8W_1%
Connections:
- net V_Qwiic is gone; now on net VIN: JP1.2 (B), JP2.2 (B), R2.2, R3.1, U1.5 (VS)
- net GND: now also U2.12 (GND), JP7.1 (A), R6.2, R7.2, R8.2
- net SC0: now also R5.2
- net SD0: now also R4.2
- net at U2.1 (A0): now also R8.1
- net SD3: now reaches U2.10 (SD3)
- net SC3: now reaches U2.11 (SC3)
- net SD4: now reaches U2.13 (SD4)
- net SC4: now reaches U2.14 (SC4)
- net SD5: now reaches U2.15 (SD5)
- net SC5: now reaches U2.16 (SC5)
- net SD6: now reaches U2.17 (SD6)
- net SC6: now reaches U2.18 (SC6)
- net SD7: now reaches U2.19 (SD7)
- net at U2.2 (A1): now also JP6.2 (B), R7.1
- net SC7: now reaches U2.20 (SC7)
- net at U2.21 (A2): now also JP5.1 (A), R6.1
- net at U2.22 (SCL): now also JP4.1 (A)
- net at U2.23 (SDA): now also JP3.1 (A)
- net VIN: now reaches U2.24 (VCC)
- net VIN: now also U2.3 (RESET#), JP5.2 (B), JP6.1 (A), JP7.2 (B)
- net SD1: now reaches U2.6 (SD1)
- net SC1: now reaches U2.7 (SC1)
- net SD2: now reaches U2.8 (SD2)
- net SC2: now reaches U2.9 (SC2)
- new net: JP3.2 (B), R4.1
- new net: JP4.2 (B), R5.1
Other:
- note added: "Cut JP3 and JP4 to disable pullups"
- note added: "Solar Cell JST Connections"
- moved on the sheet: J1, J10, J11, J12, J2, J3, J4, J5, J6, J7, J8, J9

Commit message: worked on schematic
Parts:
- added C1: 10 uF, power_board_footprints_V2.0:C_0603, symbol power_board_symbols_V2.0:C_10uF_0603
- added C2, C3: 4.7 uF, power_board_footprints_V2.0:C_0603, symbol power_board_symbols_V2.0:C_4.7uF_0603
- added D10, D12, D4, D6, D8: 20V 1A, Diode_SMD:D_SOD-323, symbol power_board_symbols_V2.0:D_Schottky_20V_1A_SOD-323
- added D11, D3, D5, D7, D9: 1W 6.2V, power_board_footprints_V2.0:Z_DO-214AC, symbol power_board_symbols_V2.0:Z_1W_6.2V_DO-214AC
- added J13, J14: ~, power_board_footprints_V2.0:QWIIC_CONN_RA, symbol power_board_symbols_V2.0:QWIIC_CONNECTOR_RA
- added JP10, JP11, JP12, JP13, JP14, JP15, JP16, JP17, JP8, JP9: SolderJumper_2_Open, Jumper:SolderJumper-2_P1.3mm_Open_RoundedPad1.0x1.5mm, symbol Jumper:SolderJumper_2_Open
- added LED1: ~, power_board_footprints_V2.0:LED_0603, symbol power_board_symbols_V2.0:LED_0603
- added LOGO1: ~, power_board_footprints_V2.0:OSHW-LOGO-L, symbol power_board_symbols_V2.0:OSHW-LOGOL
- added LOGO2: ~, power_board_footprints_V2.0:QWIIC_logo_8MM, symbol power_board_symbols_V2.0:QWIIC_LOGO_8MM
- added R10, R11, R13, R14, R16, R17, R19, R20, R22, R23: 10 kOhm, power_board_footprints_V2.0:R_0805, symbol power_board_symbols_V2.0:R_10kOhm_1/8W_1%
- added R12, R15, R18, R21, R9: 100 mOhm, power_board_footprints_V2.0:R_shunt, symbol power_board_symbols_V2.0:R_shunt_100mOhm_2W_1%
- added R24: 4.7 kOhm, power_board_footprints_V2.0:R_0603, symbol power_board_symbols_V2.0:R_4.7kOhm_0603
- added R25: 2 kOhm, power_board_footprints_V2.0:R_0603, symbol power_board_symbols_V2.0:R_2kOhm_0603
- added U3, U4, U5, U6, U7: INA219AIDR, power_board_footprints_V2.0:INA219AIDR, symbol power_board_symbols_V2.0:INA219AIDR
- added U8: MCP73831T-2ACI/OT, power_board_footprints_V2.0:MCP73831_IC_BATT_CNTL, symbol power_board_symbols_V2.0:MCP73831_IC_BATT_CNTL
Connections:
- net SC1 is gone; now on net SC0: U2.7 (SC1)
- net SC2 is gone; now on net SC0: U2.9 (SC2)
- net SC3 is gone; now on net SC0: U2.11 (SC3)
- net SC4 is gone; now on net SC0: U2.14 (SC4)
- net SC5 is gone; now on net SC0: U2.16 (SC5)
- net SD1 is gone; now on net SD0: U2.6 (SD1)
- net SD2 is gone; now on net SD0: U2.8 (SD2)
- net SD4 is gone; now on net SD0: U2.13 (SD4)
- net SD5 is gone; now on net SD0: U2.15 (SD5)
- net +Y_IN+: now also R12.2, U4.8 (VIN+)
- net +Y_IN-: now also D5.2, D6.2 (A), R12.1, U4.7 (VIN-)
- net +Z_IN+: now also R18.2, U6.8 (VIN+)
- net +Z_IN-: now also D10.2 (A), D9.2, R18.1, U6.7 (VIN-)
- net -X_IN+: now also R9.2, U3.8 (VIN+)
- net -X_IN-: now also D3.2, D4.2 (A), R9.1, U3.7 (VIN-)
- net -Y_IN+: now also R15.2, U5.8 (VIN+)
- net -Y_IN-: now also D7.2, D8.2 (A), R15.1, U5.7 (VIN-)
- net -Z_IN+: now also R21.2, U7.8 (VIN+)
- net -Z_IN-: now also D11.2, D12.2 (A), R21.1, U7.7 (VIN-)
- net GND: now also C1.1, C2.1, C3.1, J13.1, J14.1, R10.1, R11.2, R13.1, R14.2, R16.1, R17.2, R19.1, R20.2, R22.1, R23.2, R25.1, U3.6 (GND), U4.6 (GND), U5.6 (GND), U6.6 (GND), U7.6 (GND), U8.2 (VSS)
- net IN-: now also C2.2, D10.1 (K), D11.1, D12.1 (K), D3.1, D4.1 (K), D5.1, D6.1 (K), D7.1, D8.1 (K), D9.1, R24.1, U8.4 (VDD)
- net SC0: now also J13.4, J14.4, U3.4 (SCL), U4.4 (SCL), U5.4 (SCL), U6.4 (SCL), U7.4 (SCL)
- net SD0: now also J13.3, J14.3, U3.3 (SDA), U4.3 (SDA), U5.3 (SDA), U6.3 (SDA), U7.3 (SDA)
- net VIN: now also C1.2, J13.2, J14.2, JP10.2 (B), JP11.2 (B), JP12.2 (B), JP13.2 (B), JP14.2 (B), JP15.2 (B), JP16.2 (B), JP17.2 (B), JP8.2 (B), JP9.2 (B), R10.2, R11.1, R13.2, R14.1, R16.2, R17.1, R19.2, R20.1, R22.2, R23.1, U3.5 (VS), U4.5 (VS), U5.5 (VS), U6.5 (VS), U7.5 (VS)
- new net: JP14.1 (A), U6.1 (A1)
- new net: JP15.1 (A), U6.2 (A0)
- new net: LED1.1 (-), U8.1 (STAT)
- new net: R25.2, U8.5 (PROG)
- new net: JP17.1 (A), U7.2 (A0)
- new net: JP10.1 (A), U4.1 (A1)
- new net: JP11.1 (A), U4.2 (A0)
- new net: LED1.2 (+), R24.2
- new net: JP8.1 (A), U3.1 (A1)
- new net: JP9.1 (A), U3.2 (A0)
- new net: JP12.1 (A), U5.1 (A1)
- new net: JP13.1 (A), U5.2 (A0)
- new net: JP16.1 (A), U7.1 (A1)
- new net V_BATT: C3.2, U8.3 (VBAT)
Other:
- note added: "Circuit design from: https://github.com/adafruit/Adafruit-TCA9548A-I2C-Multiplexer-PCB"
- moved on the sheet: JP3, JP4, JP5, JP6, JP7, R4, R5, R6, R7, R8, U2

Commit message: work on pcb positioning
Parts:
- added D13: 1W 6.2V, power_board_footprints_V2.0:Z_DO-214AC, symbol power_board_symbols_V2.0:Z_1W_6.2V_DO-214AC
- added D14: 20V 1A, Diode_SMD:D_SOD-323, symbol power_board_symbols_V2.0:D_Schottky_20V_1A_SOD-323
- added H1, H2: MountingHole_Pad, power_board_footprints_V2.0:MountingHole_3.2mm_Pad_Oval, symbol power_board_symbols_V2.0:MountingHole_Pad
- added H3, H4: MountingHole_Pad, MountingHole:MountingHole_3.2mm_M3_Pad, symbol power_board_symbols_V2.0:MountingHole_Pad
- added J15, J16: CONN 2MM JST, power_board_footprints_V2.0:CONN_2mm_JST, symbol power_board_symbols_V2.0:CONN 2mm JST
- added JP18, JP19: SolderJumper_2_Open, Jumper:SolderJumper-2_P1.3mm_Open_RoundedPad1.0x1.5mm, symbol Jumper:SolderJumper_2_Open
- added R26: 100 mOhm, power_board_footprints_V2.0:R_shunt, symbol power_board_symbols_V2.0:R_shunt_100mOhm_2W_1%
- added R27, R28: 10 kOhm, power_board_footprints_V2.0:R_0805, symbol power_board_symbols_V2.0:R_10kOhm_1/8W_1%
- added TP1, TP2, TP3, TP4, TP5, TP6, TP7, TP8: ~, power_board_footprints_V2.0:1X02_NO_SILK, symbol power_board_symbols_V2.0:CONN_021X02_NO_SILK
- added U8: INA219AIDR, power_board_footprints_V2.0:INA219AIDR, symbol power_board_symbols_V2.0:INA219AIDR
- renumbered J11 to J10, J9 to J11, J10 to J8, J8 to J9, U3 to U2, U4 to U3, U5 to U4, U6 to U5, U7 to U6, U2 to U7, U8 to U9
Connections:
- net SC6 is gone; now on net SC0: U7.18 (SC6)
- net SD3 is gone; now on net SD0: U7.10 (SD3)
- net SD6 is gone; now on net SD0: U7.17 (SD6)
- net +X_IN+: now also TP1.2
- net +X_IN-: no longer J1.1, J2.1
- net +Y_IN+: now also TP3.2
- net +Y_IN-: no longer J5.1, J6.1
- net +Z_IN+: now also TP5.2
- net +Z_IN-: no longer J10.1, J9.1
- net -X_IN+: now also TP2.2
- net -X_IN-: no longer J3.1, J4.1
- net -Y_IN+: now also TP4.2
- net -Y_IN-: no longer J7.1, J8.1
- net -Z_IN+: now also TP6.2
- net -Z_IN-: no longer J11.1, J12.1
- net GND: now also J1.1, J10.1, J11.1, J12.1, J2.1, J3.1, J4.1, J5.1, J6.1, J7.1, J8.1, J9.1, H1.1, H2.1, H3.1, H4.1, J15.2, J15.3 (SHIELD), J15.4 (SHIELD), J16.1, J16.3 (SHIELD), J16.4 (SHIELD), R27.1, R28.2, TP1.1, TP2.1, TP3.1, TP4.1, TP5.1, TP6.1, TP7.1, TP8.1, U8.6 (GND)
- net SC0: now also U8.4 (SCL)
- net SD0: now also U8.3 (SDA)
- net VIN: now also JP18.2 (B), JP19.2 (B), R27.2, R28.1, U8.5 (VS)
- net V_BATT: now also J15.1, R26.2, TP8.2, U8.8 (VIN+)
- net IN- renamed solar_IN
- net solar_IN: now also TP7.2
- new net: D13.2, D14.2 (A), R26.1, U8.7 (VIN-)
- new net: JP19.1 (A), U8.2 (A0)
- new net: JP18.1 (A), U8.1 (A1)
- new net Batt_OUT: D13.1, D14.1 (K), J16.2
Other:
- note added: "Battery DC Current Sensor"
- note added: "Battery Input"
- note added: "Battery JST Connectors"
- note added: "Battery Output (To Main Board)"
- note added: "I2C Multiplexer"
- note added: "LiPo Battery Charger"
- note added: "Qwiic Connections"
- note added: "Solar Cell DC Current Sensors"
- note added: "Test pads"
- moved on the sheet: C1, C2, C3, D1, D10, D11, D12, D2, D3, D4, D5, D6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

Commit message: routing work
Parts:
- removed JP1, JP10, JP11, JP12, JP13, JP14, JP15, JP16, JP17, JP18, JP19, JP2, JP8, JP9: SolderJumper_2_Open, Jumper:SolderJumper-2_P1.3mm_Open_RoundedPad1.0x1.5mm, symbol Jumper:SolderJumper_2_Open
- removed R10, R11, R13, R14, R16, R17, R19, R2, R20, R22, R23, R27, R28, R3: 10 kOhm, power_board_footprints_V2.0:R_0805, symbol power_board_symbols_V2.0:R_10kOhm_1/8W_1%
- added LOGO3: ~, power_board_footprints_V2.0:QWIIC_logo_8MM, symbol power_board_symbols_V2.0:QWIIC_LOGO_8MM
Connections:
- net SC0: no longer J13.4, J14.4, R5.2, U2.4 (SCL), U3.4 (SCL), U4.4 (SCL), U5.4 (SCL), U6.4 (SCL), U7.11 (SC3), U7.14 (SC4), U7.16 (SC5), U7.18 (SC6), U7.7 (SC1), U7.9 (SC2), U8.4 (SCL)
- net SD0: no longer J13.3, J14.3, R4.2, U2.3 (SDA), U3.3 (SDA), U4.3 (SDA), U5.3 (SDA), U6.3 (SDA), U7.10 (SD3), U7.13 (SD4), U7.15 (SD5), U7.17 (SD6), U7.6 (SD1), U7.8 (SD2), U8.3 (SDA)
- new net SC1: U2.4 (SCL), U7.7 (SC1)
- new net SC2: U3.4 (SCL), U7.9 (SC2)
- new net SC3: U4.4 (SCL), U7.11 (SC3)
- new net SC4: U5.4 (SCL), U7.14 (SC4)
- new net SC5: U6.4 (SCL), U7.16 (SC5)
- new net SC6: U7.18 (SC6), U8.4 (SCL)
- new net SCL: J13.4, J14.4, R5.2
- new net SD1: U2.3 (SDA), U7.6 (SD1)
- new net SD2: U3.3 (SDA), U7.8 (SD2)
- new net SD3: U4.3 (SDA), U7.10 (SD3)
- new net SD4: U5.3 (SDA), U7.13 (SD4)
- new net SD5: U6.3 (SDA), U7.15 (SD5)
- new net SD6: U7.17 (SD6), U8.3 (SDA)
- new net SDA: J13.3, J14.3, R4.2
- no-connect marks 0 -> 14

Commit message: finished v2.0
Other:
- note added: "I2C Address: 0x70"
Changed lines of the file:
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@@
+		)
+	)
+	(text "I2C Address: 0x70"
+		(exclude_from_sim no)
+		(at 353.822 138.176 0)
+		(effects
+			(font
+				(size 1.27 1.27)
+			)
 		)
 	)

Commit message: Updated to replace out of stock comps.
Zener diodes were out of stock with JLCPCB. Updated production folder to include replacement components.
Parts:
- D11, D13, D2, D3, D5, D7, D9: LCSC C110527 -> C151039
Changed lines of the file:
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@@
 			)
 		)
-		(property "Datasheet" "https://jlcpcb.com/api/file/downloadByFileSystemAccessId/8560078683311935488"
+		(property "Datasheet" "https://jlcpcb.com/api/file/downloadByFileSystemAccessId/8588880030219190272"
 			(at 328.803 72.136 0)
 			(effects
@@
 			)
 		)
-		(property "Description" "https://jlcpcb.com/partdetail/DiodesIncorporated-SMAZ6V2_13F/C110527"
+		(property "Description" "https://jlcpcb.com/partdetail/DiodesIncorporated-SMAZ6V8_13F/C151039"
 			(at 328.93 69.85 0)
 			(effects
@@
 			)
 		)
-		(property "LCSC" "C110527"
+		(property "LCSC" "C151039"
 			(at 328.93 69.85 0)
 			(effects
@@
 			)
 		)
-		(property "Datasheet" "https://jlcpcb.com/api/file/downloadByFileSystemAccessId/8560078683311935488"
+		(property "Datasheet" "https://jlcpcb.com/api/file/downloadByFileSystemAccessId/8588880030219190272"
 			(at 222.123 163.576 0)
 			(effects
@@
 			)
 		)
-		(property "Description" "https://jlcpcb.com/partdetail/DiodesIncorporated-SMAZ6V2_13F/C110527"
+		(property "Description" "https://jlcpcb.com/partdetail/DiodesIncorporated-SMAZ6V8_13F/C151039"
 			(at 222.25 161.29 0)
 			(effects
@@
 			)
 		)
-		(property "LCSC" "C110527"
+		(property "LCSC" "C151039"
 			(at 222.25 161.29 0)
 			(effects
@@
 			)
 		)
-		(property "Datasheet" "https://jlcpcb.com/api/file/downloadByFileSystemAccessId/8560078683311935488"
+		(property "Datasheet" "https://jlcpcb.com/api/file/downloadByFileSystemAccessId/8588880030219190272"
 			(at 222.123 67.056 0)
 			(effects
@@
 			)
 		)
-		(property "Description" "https://jlcpcb.com/partdetail/DiodesIncorporated-SMAZ6V2_13F/C110527"
+		(property "Description" "https://jlcpcb.com/partdetail/DiodesIncorporated-SMAZ6V8_13F/C151039"
 			(at 222.25 64.77 0)
 			(effects
@@
 			)
 		)
-		(property "LCSC" "C110527"
+		(property "LCSC" "C151039"
 			(at 222.25 64.77 0)
 			(effects
@@
 			)
 		)
-		(property "Datasheet" "https://jlcpcb.com/api/file/downloadByFileSystemAccessId/8560078683311935488"
+		(property "Datasheet" "https://jlcpcb.com/api/file/downloadByFileSystemAccessId/8588880030219190272"
 			(at 145.923 67.056 0)
 			(effects
@@
 			)
 		)
-		(property "Description" "https://jlcpcb.com/partdetail/DiodesIncorporated-SMAZ6V2_13F/C110527"
+		(property "Description" "https://jlcpcb.com/partdetail/DiodesIncorporated-SMAZ6V8_13F/C151039"
 			(at 146.05 64.77 0)
 			(effects
@@
 			)
 		)
-		(property "LCSC" "C110527"
+		(property "LCSC" "C151039"
 			(at 146.05 64.77 0)
 			(effects
@@
 			)
 		)
-		(property "Datasheet" "https://jlcpcb.com/api/file/downloadByFileSystemAccessId/8560078683311935488"
+		(property "Datasheet" "https://jlcpcb.com/api/file/downloadByFileSystemAccessId/8588880030219190272"
 			(at 222.123 114.046 0)
 			(effects
@@
 			)
 		)
-		(property "Description" "https://jlcpcb.com/partdetail/DiodesIncorporated-SMAZ6V2_13F/C110527"
+		(property "Description" "https://jlcpcb.com/partdetail/DiodesIncorporated-SMAZ6V8_13F/C151039"
 			(at 222.25 111.76 0)
 			(effects
@@
 			)
 		)
-		(property "LCSC" "C110527"
+		(property "LCSC" "C151039"
 			(at 222.25 111.76 0)
 			(effects
@@
 			)
 		)
-		(property "Datasheet" "https://jlcpcb.com/api/file/downloadByFileSystemAccessId/8560078683311935488"
+		(property "Datasheet" "https://jlcpcb.com/api/file/downloadByFileSystemAccessId/8588880030219190272"
 			(at 145.923 114.046 0)
 			(effects
@@
 			)
 		)
-		(property "Description" "https://jlcpcb.com/partdetail/DiodesIncorporated-SMAZ6V2_13F/C110527"
+		(property "Description" "https://jlcpcb.com/partdetail/DiodesIncorporated-SMAZ6V8_13F/C151039"
 			(at 146.05 111.76 0)
 			(effects
@@
 			)
 		)
-		(property "LCSC" "C110527"
+		(property "LCSC" "C151039"
 			(at 146.05 111.76 0)
 			(effects
@@
 			)
 		)
-		(property "Datasheet" "https://jlcpcb.com/api/file/downloadByFileSystemAccessId/8560078683311935488"
+		(property "Datasheet" "https://jlcpcb.com/api/file/downloadByFileSystemAccessId/8588880030219190272"
 			(at 145.923 163.576 0)
 			(effects
@@
 			)
 		)
-		(property "Description" "https://jlcpcb.com/partdetail/DiodesIncorporated-SMAZ6V2_13F/C110527"
+		(property "Description" "https://jlcpcb.com/partdetail/DiodesIncorporated-SMAZ6V8_13F/C151039"
 			(at 146.05 161.29 0)
 			(effects
@@
 			)
 		)
-		(property "LCSC" "C110527"
+		(property "LCSC" "C151039"
 			(at 146.05 161.29 0)
 			(effects
